File: Projeto VBS.kicad_pcb (KiCad board)
At the start: 2 copper layers, 6 parts, among them J1_tx/rx1 Conn_01x03_Pin, J2_fins_de_curso1 Conn_01x03_Pin, J3 Conn_01x03_Pin, J4 Conn_01x06_Pin, J5 Conn_01x02_Socket

Commit message: falta a malha de negativo
Parts:
- added LM2596Module1: ~, lm2597:LM2596 Module, F.Cu at (136.5, 139.5)
- moved J1_tx/rx1 71.6 mm to (100.5, 77.0)
- moved A1 68.8 mm to (126.0, 96.0)
- moved J3 60.0 mm to (150.5, 108.0), turned to 90 degrees
- moved J5 51.2 mm to (100.0, 141.0), turned to 90 degrees
- moved J2_fins_de_curso1 39.7 mm to (100.5, 93.5), turned to -90 degrees
- moved J4 2.28 mm to (100.3, 110.2), turned to -90 degrees
Connections:
- A1 pad 16: unconnected-(A1-GPIO12-Pad16) -> Net-(A1-GPIO12)
- A1 pad 40: unconnected-(A1-VBUS-Pad40) -> Net-(A1-VBUS)
- J4 pad 1: unconnected-(J4-Pin_1-Pad1) -> Net-(J4-Pin_1)
- J4 pad 2: unconnected-(J4-Pin_2-Pad2) -> Net-(J4-Pin_2)
- J4 pad 4: unconnected-(J4-Pin_4-Pad4) -> Net-(A1-GPIO12)
- J5 pad 1: unconnected-(J5-Pin_1-Pad1) -> Net-(J4-Pin_2)
- J5 pad 2: unconnected-(J5-Pin_2-Pad2) -> Net-(J4-Pin_1)
Routing:
- net Net-(A1-3V3_EN): track 0.00 -> 101.8 mm
- net Net-(A1-VBUS): track 0.00 -> 99.0 mm
- net Net-(J1_tx/rx1-Pin_1): track 0.00 -> 59.3 mm
- net Net-(J4-Pin_2): track 0.00 -> 55.9 mm
- net Net-(J4-Pin_1): track 0.00 -> 54.6 mm
- net Net-(A1-GPIO4): track 0.00 -> 20.5 mm
- net Net-(A1-GPIO5): track 0.00 -> 20.5 mm
- net Net-(A1-GPIO26_ADC0): track 0.00 -> 18.2 mm
- net Net-(A1-GPIO3): track 0.00 -> 15.8 mm
- net Net-(A1-GPIO2): track 0.00 -> 15.8 mm
Other:
- board outline added: 120 x 120 mm

Commit message: placa quase pronta
Parts:
- removed J5: Conn_01x02_Socket, Connector_AMASS:AMASS_XT30UPB-F_1x02_P5.0mm_Vertical
- added J1: Screw_Terminal_01x02, TerminalBlock_Phoenix:TerminalBlock_Phoenix_PT-1,5-2-5.0-H_1x02_P5.00mm_Horizontal, B.Cu at (100.0, 137.2)
Connections:
- A1 pad 13: Net-(J1_tx/rx1-Pin_1) -> GND
- A1 pad 18: Net-(J1_tx/rx1-Pin_1) -> GND
- A1 pad 23: Net-(J1_tx/rx1-Pin_1) -> GND
- A1 pad 28: Net-(J1_tx/rx1-Pin_1) -> GND
- A1 pad 3: Net-(J1_tx/rx1-Pin_1) -> GND
- A1 pad 38: Net-(J1_tx/rx1-Pin_1) -> GND
- A1 pad 8: Net-(J1_tx/rx1-Pin_1) -> GND
- J1_tx/rx1 pad 1: Net-(J1_tx/rx1-Pin_1) -> GND
- J3 pad 2: Net-(J1_tx/rx1-Pin_1) -> GND
- J4 pad 2: Net-(J4-Pin_2) -> GND
- LM2596Module1 pad 2: Net-(J4-Pin_2) -> GND
- LM2596Module1 pad 4: Net-(J1_tx/rx1-Pin_1) -> GND
Routing:
- net Net-(J1_tx/rx1-Pin_1): track 59.3 -> 0.00 mm
- net Net-(J4-Pin_2): track 55.9 -> 0.00 mm
- net Net-(A1-GPIO12): track 0.00 -> 19.2 mm
- net Net-(A1-3V3_EN): track 101.8 -> 110.1 mm
- net Net-(J1-Pin_1): track 54.6 -> 55.6 mm
- added copper zone on B.Cu, net GND

Commit message: acho que esta pronto
Parts:
- J1_tx/rx1: footprint Connector_JST:JST_XH_S3B-XH-A-1_1x03_P2.50mm_Horizontal -> Connector_JST:JST_XH_B3B-XH-A_1x03_P2.50mm_Vertical; moved to B.Cu
- J2_fins_de_curso1, J3: footprint Connector_JST:JST_XH_S3B-XH-A-1_1x03_P2.50mm_Horizontal -> Connector_JST:JST_XH_B3B-XH-A_1x03_P2.50mm_Vertical
- J4: footprint Connector_JST:JST_XH_S6B-XH-A-1_1x06_P2.50mm_Horizontal -> Connector_JST:JST_XH_B6B-XH-A_1x06_P2.50mm_Vertical
- moved J1 80.2 mm to (152.0, 76.2)
- moved LM2596Module1 59.0 mm to (125.2, 81.6), turned to 180 degrees
- moved J4 53.5 mm to (131.9, 67.0), turned to 180 degrees
- moved J3 53.4 mm to (97.8, 116.5), turned to -90 degrees
- moved J1_tx/rx1 53.1 mm to (152.0, 89.8)
- moved A1 16.7 mm to (130.1, 112.2), turned to -90 degrees
- moved J2_fins_de_curso1 9.97 mm to (97.8, 103.1)
Routing:
- net Net-(A1-3V3_EN): track 110.1 -> 77.7 mm
- net Net-(J1-Pin_1): track 55.6 -> 23.9 mm
- net Net-(A1-GPIO4): track 20.5 -> 52.1 mm
- net Net-(A1-GPIO5): track 20.5 -> 50.2 mm
- net Net-(A1-VBUS): track 98.5 -> 121.7 mm
- net Net-(A1-GPIO12): track 19.2 -> 39.8 mm, vias 0 -> 2
- net Net-(A1-GPIO26_ADC0): track 18.2 -> 35.6 mm
- net Net-(A1-GPIO3): track 15.8 -> 12.3 mm
- net Net-(A1-GPIO2): track 15.8 -> 17.2 mm
Other:
- board size 120 x 120 mm -> 65.8 x 66.1 mm
