File: Projeto VBS.kicad_sch (KiCad schematic)
At the start: 6 parts, among them J1_tx/rx1 Conn_01x03_Pin, J2_fins_de_curso1 Conn_01x03_Pin, J3 Conn_01x03_Pin, J4 Conn_01x06_Pin, J5 Conn_01x02_Socket

Commit message: falta a malha de negativo
Parts:
- added LM2596Module1: ~, lm2597:LM2596 Module, symbol lm2597:lm2597
Connections:
- net at A1.13 (GND), A1.18 (GND), A1.23 (GND)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: now also LM2596Module1.4 (Vout-)
- net at J5.1 (Pin_1): now also J4.2 (Pin_2), LM2596Module1.2 (Vin-)
- net at J5.2 (Pin_2): now also J4.1 (Pin_1), LM2596Module1.1 (Vin+)
- net at A1.16 (GPIO12): now also J4.4 (Pin_4)
- net at A1.40 (VBUS): now also LM2596Module1.3 (Vout+)
Other:
- moved on the sheet: J4, J5

Commit message: placa quase pronta
Parts:
- removed J5: Conn_01x02_Socket, Connector_AMASS:AMASS_XT30UPB-F_1x02_P5.0mm_Vertical, symbol Connector:Conn_01x02_Socket
- added J1: Screw_Terminal_01x02, TerminalBlock_Phoenix:TerminalBlock_Phoenix_PT-1,5-2-5.0-H_1x02_P5.00mm_Horizontal, symbol Connector:Screw_Terminal_01x02
- LM2596Module1: value ~ -> (none)
Connections:
- net GND: now reaches A1.13 (GND), A1.18 (GND), A1.23 (GND), A1.28 (GND), A1.3 (GND), A1.38 (GND), A1.8 (GND), J1_tx/rx1.1 (Pin_1), J3.2 (Pin_2), LM2596Module1.4 (Vout-)
- net GND: now also J4.2 (Pin_2), LM2596Module1.2 (Vin-), J1.2 (Pin_2)
- net at J4.1 (Pin_1), LM2596Module1.1 (Vin+): now also J1.1 (Pin_1)

Commit message: acho que esta pronto 2
Parts:
- J1_tx/rx1, J2_fins_de_curso1, J3: footprint Connector_JST:JST_XH_S3B-XH-A-1_1x03_P2.50mm_Horizontal -> Connector_JST:JST_XH_B3B-XH-A_1x03_P2.50mm_Vertical
- J4: footprint Connector_JST:JST_XH_S6B-XH-A-1_1x06_P2.50mm_Horizontal -> Connector_JST:JST_XH_B6B-XH-A_1x06_P2.50mm_Vertical
Connections:
- net at A1.6 (GPIO4): now also J2_fins_de_curso1.3 (Pin_3); no longer J2_fins_de_curso1.2 (Pin_2)
- net at A1.7 (GPIO5): now also J2_fins_de_curso1.2 (Pin_2); no longer J2_fins_de_curso1.3 (Pin_3)
Changed lines of the file:
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@@
 	(wire
 		(pts
-			(xy 137.16 49.53) (xy 100.33 49.53)
+			(xy 100.33 49.53) (xy 139.7 49.53)
 		)
 		(stroke
@@
 	(wire
 		(pts
-			(xy 137.16 46.99) (xy 137.16 49.53)
-		)
-		(stroke
-			(width 0)
-			(type default)
-		)
-	)
-	(wire
-		(pts
 			(xy 161.29 52.07) (xy 161.29 46.99)
 		)
@@
 	(wire
 		(pts
-			(xy 139.7 46.99) (xy 139.7 50.8)
+			(xy 137.16 46.99) (xy 137.16 50.8)
 		)
 		(stroke
@@
 	(wire
 		(pts
+			(xy 137.16 50.8) (xy 99.06 50.8)
+		)
+		(stroke
+			(width 0)
+			(type default)
+		)
+	)
+	(wire
+		(pts
 			(xy 146.05 71.12) (xy 151.13 71.12)
 		)
@@
 	(wire
 		(pts
+			(xy 139.7 49.53) (xy 139.7 46.99)
+		)
+		(stroke
+			(width 0)
+			(type default)
+		)
+	)
+	(wire
+		(pts
 			(xy 110.49 120.65) (xy 180.34 120.65)
 		)
@@
 		(pts
 			(xy 153.67 80.01) (xy 153.67 57.15)
-		)
-		(stroke
-			(width 0)
-			(type default)
-		)
-	)
-	(wire
-		(pts
-			(xy 139.7 50.8) (xy 99.06 50.8)
 		)
 		(stroke
@@
 			)
 		)
-		(property "Footprint" "Connector_JST:JST_XH_S3B-XH-A-1_1x03_P2.50mm_Horizontal"
+		(property "Footprint" "Connector_JST:JST_XH_B3B-XH-A_1x03_P2.50mm_Vertical"
 			(at 158.75 41.91 0)
-			(hide yes)
 			(show_name no)
 			(do_not_autoplace no)
@@
 			)
 		)
-		(property "Footprint" "Connector_JST:JST_XH_S3B-XH-A-1_1x03_P2.50mm_Horizontal"
+		(property "Footprint" "Connector_JST:JST_XH_B3B-XH-A_1x03_P2.50mm_Vertical"
 			(at 24.13 60.96 0)
 			(hide yes)
@@
 			)
 		)
-		(property "Footprint" "Connector_JST:JST_XH_S6B-XH-A-1_1x06_P2.50mm_Horizontal"
+		(property "Footprint" "Connector_JST:JST_XH_B6B-XH-A_1x06_P2.50mm_Vertical"
 			(at 177.8 73.66 0)
 			(hide yes)
@@
 			)
 		)
-		(property "Footprint" "Connector_JST:JST_XH_S3B-XH-A-1_1x03_P2.50mm_Horizontal"
+		(property "Footprint" "Connector_JST:JST_XH_B3B-XH-A_1x03_P2.50mm_Vertical"
 			(at 139.7 41.91 0)
 			(hide yes)
